Commit message: Added sensors to mobile_base urdf and setup robot_state_publisher launch file.

File: urdf/mobile_base.urdf (robot description, URDF)
Before this commit: robot mobile_base, 5 links, 4 joints
Links:
- added link ir_center; visual box size=.0014 0.0030 0.0013
- added link ir_left; visual box size=.0014 0.0030 0.0013
- added link ir_right; visual box size=.0014 0.0030 0.0013
- added link sonar_left; visual box size=.0015 0.0046 0.0021
- added link sonar_right; visual box size=.0015 0.0046 0.0021
Joints:
- added joint ir_center_joint: type fixed, parent platform, child ir_center, origin xyz=0.1023 0 0.005 rpy=0 0 0
- added joint ir_left_joint: type fixed, parent platform, child ir_left, origin xyz=0.0766 -0.125 0.005 rpy=0 0 -0.7
- added joint ir_right_joint: type fixed, parent platform, child ir_right, origin xyz=0.0766 0.125 0.005 rpy=0 0 0.7
- added joint sonar_left_joint: type fixed, parent platform, child sonar_left, origin xyz=0.0936 -0.0635 0.005 rpy=0 0 -0.35
- added joint sonar_right_joint: type fixed, parent platform, child sonar_right, origin xyz=0.0936 0.0635 0.005 rpy=0 0 0.35

File: urdf/mobile_base.xacro (robot description, xacro)
@@ -8,4 +8,5 @@
   <xacro:property name="wheel_w_offset" value=".0025" />
   <xacro:property name="wheel_h_offset" value="-.015" />
+  <xacro:property name="sensor_height" value="0.0050" />
   <xacro:property name="pi" value="3.14159265359" />
   <!-- fictitious center point on ground and between wheels for navigation -->
@@ -31,4 +32,10 @@
     </visual>
   </link>
+  <joint name="base_footprint_joint" type="fixed">
+    <parent link="base_footprint" />
+    <child link="base_link" />
+    <origin xyz="0 0 ${wheel_r}" rpy="0 0 0" />
+  </joint>
+  <!-- Base platform -->
   <link name="platform">
     <visual>
@@ -41,31 +48,4 @@
     </visual>
   </link>
-  <link name="wheel_left">
-    <visual>
-      <geometry>
-        <cylinder radius="${wheel_r}" length="${wheel_l}" />
-      </geometry>
-      <origin rpy="${pi / 2} 0 0" />
-      <material name="black">
-        <color rgba="0 0 0 1" />
-      </material>
-    </visual>
-  </link>
-  <link name="wheel_right">
-    <visual>
-      <geometry>
-        <cylinder radius="${wheel_r}" length="${wheel_l}" />
-      </geometry>
-      <origin rpy="${(pi / 2) * -1} 0 0" />
-      <material name="black">
-        <color rgba="0 0 0 1" />
-      </material>
-    </visual>
-  </link>
-  <joint name="base_footprint_joint" type="fixed">
-    <parent link="base_footprint" />
-    <child link="base_link" />
-    <origin xyz="0 0 ${wheel_r}" rpy="0 0 0" />
-  </joint>
   <joint name="platform_joint" type="fixed">
     <parent link="base_link" />
@@ -73,15 +53,65 @@
     <origin xyz="0 0 ${wheel_r + wheel_h_offset}" rpy="0 0 0" />
   </joint>
-  <joint name="wheel_left_joint" type="continuous">
-    <parent link="base_link" />
-    <child link="wheel_left" />
-    <axis xyz="0 1 0" />
-    <origin rpy="0 0 0" xyz="0 ${(platform_w / 2) + (wheel_l / 2) + wheel_w_offset} 0" />
-  </joint>
-  <joint name="wheel_right_joint" type="continuous">
-    <parent link="base_link" />
-    <child link="wheel_right" />
-    <axis xyz="0 1 0" />
-    <origin rpy="0 0 0" xyz="0 ${((platform_w / 2) + (wheel_l / 2) + wheel_w_offset) * -1} 0" />
-  </joint>
+  <!-- Differential Drive Wheels -->
+  <xacro:macro name="wheel" params="pos rpy">
+    <link name="wheel_${pos}">
+      <visual>
+        <geometry>
+          <cylinder radius="${wheel_r}" length="${wheel_l}" />
+        </geometry>
+        <origin rpy="${rpy}" />
+        <material name="black">
+          <color rgba="0 0 0 1" />
+        </material>
+      </visual>
+    </link>
+  </xacro:macro>
+  <xacro:wheel pos="right" rpy="${pi / 2} 0 0" />
+  <xacro:wheel pos="left" rpy="${(pi / 2) * -1} 0 0" />
+  <xacro:macro name="wheel_joint" params="pos xyz">
+    <joint name="wheel_${pos}_joint" type="continuous">
+      <parent link="base_link" />
+      <child link="wheel_${pos}" />
+      <axis xyz="0 1 0" />
+      <origin rpy="0 0 0" xyz="${xyz}" />
+    </joint>
+  </xacro:macro>
+  <xacro:wheel_joint pos="left" xyz="0 ${(platform_w / 2) + (wheel_l / 2) + wheel_w_offset} 0" />
+  <xacro:wheel_joint pos="right" xyz="0 ${((platform_w / 2) + (wheel_l / 2) + wheel_w_offset) * -1} 0" />
+  <!-- Sensor Array -->
+  <xacro:macro name="sonar" params="pos">
+    <link name="sonar_${pos}">
+      <visual>
+        <geometry>
+          <box size=".0015 0.0046 0.0021"/>
+        </geometry>
+      </visual>
+    </link>
+  </xacro:macro>
+  <xacro:sonar pos="left" />
+  <xacro:sonar pos="right" />
+  <xacro:macro name="ir" params="pos">
+    <link name="ir_${pos}">
+      <visual>
+        <geometry>
+          <box size=".0014 0.0030 0.0013"/>
+        </geometry>
+      </visual>
+    </link>
+  </xacro:macro>
+  <xacro:ir pos="left" />
+  <xacro:ir pos="center" />
+  <xacro:ir pos="right" />
+  <xacro:macro name="sensor_joint" params="sensor pos rpy xyz">
+    <joint name="${sensor}_${pos}_joint" type="fixed">
+      <parent link="platform" />
+      <child link="${sensor}_${pos}" />
+      <origin rpy="${rpy}" xyz="${xyz}" />
+    </joint>
+  </xacro:macro>
+  <xacro:sensor_joint sensor="sonar" pos="left" rpy="0 0 -0.35" xyz="${(platform_l / 2) - 0.008} -0.0635 ${sensor_height}" />
+  <xacro:sensor_joint sensor="sonar" pos="right" rpy="0 0 0.35" xyz="${(platform_l / 2) - 0.008} 0.0635 ${sensor_height}" />
+  <xacro:sensor_joint sensor="ir" pos="left" rpy="0 0 -0.7" xyz="${(platform_l / 2) - 0.025} -0.125 ${sensor_height}" />
+  <xacro:sensor_joint sensor="ir" pos="center" rpy="0 0 0" xyz="${(platform_l / 2) + 0.0007} 0 ${sensor_height}" />
+  <xacro:sensor_joint sensor="ir" pos="right" rpy="0 0 0.7" xyz="${(platform_l / 2) - 0.025} 0.125 ${sensor_height}" />
 </robot>

Commit message: Adding sensor depth frames to xacro/urdf.

File: urdf/mobile_base.urdf (robot description, URDF)
Before this commit: robot mobile_base, 10 links, 9 joints
Links:
- added link ir_center_depth_frame, mass 0.0001
- added link ir_left_depth_frame, mass 0.0001
- added link ir_right_depth_frame, mass 0.0001
- added link sonar_left_depth_frame, mass 0.0001
- added link sonar_right_depth_frame, mass 0.0001
Joints:
- added joint sensor_depth_joint: type fixed, parent ir_right, child ir_right_depth_frame, origin xyz=0 0.015 0 rpy=0 0 0

File: urdf/mobile_base.xacro (robot description, xacro)
@@ -115,3 +115,29 @@
   <xacro:sensor_joint sensor="ir" pos="center" rpy="0 0 0" xyz="${(platform_l / 2) + 0.0007} 0 ${sensor_height}" />
   <xacro:sensor_joint sensor="ir" pos="right" rpy="0 0 0.7" xyz="${(platform_l / 2) - 0.025} 0.125 ${sensor_height}" />
+  <xacro:macro name="sensor_depth_frame" params="sensor pos">
+    <link name="${sensor}_${pos}_depth_frame">
+      <inertial>
+        <mass value="0.0001" />
+        <origin xyz="0 0 0" />
+        <inertia ixx="0.0001" ixy="0.0" ixz="0.0" iyy="0.0001" iyz="0.0" izz="0.0001" />
+      </inertial>
+    </link>
+  </xacro:macro>
+  <xacro:sensor_depth_frame sensor="sonar" pos="left" />
+  <xacro:sensor_depth_frame sensor="sonar" pos="right" />
+  <xacro:sensor_depth_frame sensor="ir" pos="left" />
+  <xacro:sensor_depth_frame sensor="ir" pos="center" />
+  <xacro:sensor_depth_frame sensor="ir" pos="right" />
+  <xacro:macro name="sensor_depth_frame_joint" params="sensor pos">
+    <joint name="sensor_depth_joint" type="fixed">
+      <origin xyz="0 0.015 0" rpy="0 0 0" />
+      <parent link="${sensor}_${pos}" />
+      <child link="${sensor}_${pos}_depth_frame" />
+    </joint>
+  </xacro:macro>
+  <xacro:sensor_depth_frame_joint sensor="sonar" pos="left" />
+  <xacro:sensor_depth_frame_joint sensor="sonar" pos="right" />
+  <xacro:sensor_depth_frame_joint sensor="ir" pos="left" />
+  <xacro:sensor_depth_frame_joint sensor="ir" pos="center" />
+  <xacro:sensor_depth_frame_joint sensor="ir" pos="right" />
 </robot>

Commit message: Fixing bug in xacro naming.

File: urdf/mobile_base.urdf (robot description, URDF)
Before this commit: robot mobile_base, 15 links, 10 joints
Joints:
- removed joint sensor_depth_joint
- added joint ir_center_depth_joint: type fixed, parent ir_center, child ir_center_depth_frame, origin xyz=0 0.015 0 rpy=0 0 0
- added joint ir_left_depth_joint: type fixed, parent ir_left, child ir_left_depth_frame, origin xyz=0 0.015 0 rpy=0 0 0
- added joint ir_right_depth_joint: type fixed, parent ir_right, child ir_right_depth_frame, origin xyz=0 0.015 0 rpy=0 0 0
- added joint sonar_left_depth_joint: type fixed, parent sonar_left, child sonar_left_depth_frame, origin xyz=0 0.015 0 rpy=0 0 0
- added joint sonar_right_depth_joint: type fixed, parent sonar_right, child sonar_right_depth_frame, origin xyz=0 0.015 0 rpy=0 0 0

File: urdf/mobile_base.xacro (robot description, xacro)
@@ -130,5 +130,5 @@
   <xacro:sensor_depth_frame sensor="ir" pos="right" />
   <xacro:macro name="sensor_depth_frame_joint" params="sensor pos">
-    <joint name="sensor_depth_joint" type="fixed">
+    <joint name="${sensor}_${pos}_depth_joint" type="fixed">
       <origin xyz="0 0.015 0" rpy="0 0 0" />
       <parent link="${sensor}_${pos}" />

Commit message: urdf changes to swap left and right sensors

File: urdf/mobile_base.urdf (robot description, URDF)
Before this commit: robot mobile_base, 15 links, 14 joints
Joints:
- joint ir_left_joint: origin xyz=0.0766 -0.125 0.005 rpy=0 0 -0.7 -> xyz=0.0766 0.125 0.005 rpy=0 0 0.7
- joint ir_right_joint: origin xyz=0.0766 0.125 0.005 rpy=0 0 0.7 -> xyz=0.0766 -0.125 0.005 rpy=0 0 -0.7
- joint sonar_left_joint: origin xyz=0.0936 -0.0635 0.005 rpy=0 0 -0.35 -> xyz=0.0936 0.0635 0.005 rpy=0 0 0.35
- joint sonar_right_joint: origin xyz=0.0936 0.0635 0.005 rpy=0 0 0.35 -> xyz=0.0936 -0.0635 0.005 rpy=0 0 -0.35

File: urdf/mobile_base.xacro (robot description, xacro)
@@ -110,9 +110,9 @@
     </joint>
   </xacro:macro>
-  <xacro:sensor_joint sensor="sonar" pos="left" rpy="0 0 -0.35" xyz="${(platform_l / 2) - 0.008} -0.0635 ${sensor_height}" />
-  <xacro:sensor_joint sensor="sonar" pos="right" rpy="0 0 0.35" xyz="${(platform_l / 2) - 0.008} 0.0635 ${sensor_height}" />
-  <xacro:sensor_joint sensor="ir" pos="left" rpy="0 0 -0.7" xyz="${(platform_l / 2) - 0.025} -0.125 ${sensor_height}" />
+  <xacro:sensor_joint sensor="sonar" pos="left" rpy="0 0 0.35" xyz="${(platform_l / 2) - 0.008} 0.0635 ${sensor_height}" />
+  <xacro:sensor_joint sensor="sonar" pos="right" rpy="0 0 -0.35" xyz="${(platform_l / 2) - 0.008} -0.0635 ${sensor_height}" />
+  <xacro:sensor_joint sensor="ir" pos="left" rpy="0 0 0.7" xyz="${(platform_l / 2) - 0.025} 0.125 ${sensor_height}" />
   <xacro:sensor_joint sensor="ir" pos="center" rpy="0 0 0" xyz="${(platform_l / 2) + 0.0007} 0 ${sensor_height}" />
-  <xacro:sensor_joint sensor="ir" pos="right" rpy="0 0 0.7" xyz="${(platform_l / 2) - 0.025} 0.125 ${sensor_height}" />
+  <xacro:sensor_joint sensor="ir" pos="right" rpy="0 0 -0.7" xyz="${(platform_l / 2) - 0.025} -0.125 ${sensor_height}" />
   <xacro:macro name="sensor_depth_frame" params="sensor pos">
     <link name="${sensor}_${pos}_depth_frame">

Commit message: Removing base_footprint from xacro/urdf.

File: urdf/mobile_base.urdf (robot description, URDF)
Before this commit: robot mobile_base, 15 links, 14 joints
Links:
- removed link base_footprint
Joints:
- removed joint base_footprint_joint

File: urdf/mobile_base.xacro (robot description, xacro)
@@ -10,16 +10,5 @@
   <xacro:property name="sensor_height" value="0.0050" />
   <xacro:property name="pi" value="3.14159265359" />
-  <!-- fictitious center point on ground and between wheels for navigation -->
-  <link name="base_footprint">
-    <visual>
-      <geometry>
-        <box size="0.001 0.001 0.001" />
-      </geometry>
-      <origin xyz="0 0 0" rpy="0 0 0" />
-      <material name="black">
-        <color rgba="0 0 0 1" />
-      </material>
-    </visual>
-  </link>
+  <!-- fictitious center point between wheels for navigation -->
   <link name="base_link">
     <visual>
@@ -32,9 +21,4 @@
     </visual>
   </link>
-  <joint name="base_footprint_joint" type="fixed">
-    <parent link="base_footprint" />
-    <child link="base_link" />
-    <origin xyz="0 0 ${wheel_r}" rpy="0 0 0" />
-  </joint>
   <!-- Base platform -->
   <link name="platform">

Commit message: Added camera_link and base_camera_joint to xacro/urdf for stereo camera tf

File: urdf/mobile_base.urdf (robot description, URDF)
Before this commit: robot mobile_base, 14 links, 13 joints
Links:
- added link camera_link; visual box size=0.094 0.1168 0.071
Joints:
- added joint camera_base_link: type fixed, parent base_link, child camera_link, origin xyz=0.1016 0 0.0978 rpy=0 0 0

File: urdf/mobile_base.xacro (robot description, xacro)
@@ -37,5 +37,19 @@
     <origin xyz="0 0 ${wheel_r + wheel_h_offset}" rpy="0 0 0" />
   </joint>
-  <!-- Differential Drive Wheels -->
+  <!-- Stereo Camera -->
+  <link name="camera_link">
+    <visual>
+      <geometry>
+        <box size="0.094 0.1168 0.071 "/>
+      </geometry>
+      <material name="black" />
+    </visual>
+  </link>
+  <joint name="camera_base_link" type="fixed">
+    <parent link="base_link" />
+    <child link="camera_link" />
+    <origin xyz="${platform_l / 2} 0 ${wheel_r + wheel_h_offset + 0.080}" rpy="0 0 0" />
+  </joint>
+<!-- Differential Drive Wheels -->
   <xacro:macro name="wheel" params="pos rpy">
     <link name="wheel_${pos}">

Commit message: Adding the upper platform to the xacro/urdf and fixing the stereo camera size; along with a refactor to clean code.

File: urdf/mobile_base.urdf (robot description, URDF)
Before this commit: robot mobile_base, 15 links, 14 joints
Links:
- removed link platform
- added link platform_base; visual box size=0.2032 0.2286 0.0064
- added link platform_upper; visual box size=0.2032 0.2286 0.0064
- link camera_link: geometry visual box size=0.020 0.075 0.015
Joints:
- removed joint platform_joint
- added joint platform_joint_base: type fixed, parent base_link, child platform_base, origin xyz=0 0 0.0178 rpy=0 0 0
- added joint platform_joint_upper: type fixed, parent base_link, child platform_upper, origin xyz=0 0 0.0978 rpy=0 0 0
- joint camera_base_link: origin xyz=0.1016 0 0.0978 rpy=0 0 0 -> xyz=0.1116 0 0.0978 rpy=0 0 0
- joint ir_center_joint: parent platform -> platform_base
- joint ir_left_joint: parent platform -> platform_base
- joint ir_right_joint: parent platform -> platform_base
- joint sonar_left_joint: parent platform -> platform_base
- joint sonar_right_joint: parent platform -> platform_base

File: urdf/mobile_base.xacro (robot description, xacro)
@@ -21,25 +21,33 @@
     </visual>
   </link>
-  <!-- Base platform -->
-  <link name="platform">
-    <visual>
-      <geometry>
-        <box size="${platform_l} ${platform_w} ${platform_h}"/>
-      </geometry>
-      <material name="white">
-        <color rgba="1 1 1 1" />
-      </material>
-    </visual>
-  </link>
-  <joint name="platform_joint" type="fixed">
-    <parent link="base_link" />
-    <child link="platform" />
-    <origin xyz="0 0 ${wheel_r + wheel_h_offset}" rpy="0 0 0" />
-  </joint>
+  <!-- Bot platforms -->
+  <xacro:macro name="platform" params="pos">
+    <link name="platform_${pos}">
+      <visual>
+        <geometry>
+          <box size="${platform_l} ${platform_w} ${platform_h}"/>
+        </geometry>
+        <material name="white">
+          <color rgba="1 1 1 1" />
+        </material>
+      </visual>
+    </link>
+  </xacro:macro>
+  <xacro:platform pos="base" />
+  <xacro:platform pos="upper" />
+  <xacro:macro name="platform_joint" params="pos xyz">
+    <joint name="platform_joint_${pos}" type="fixed">
+      <parent link="base_link" />
+      <child link="platform_${pos}" />
+      <origin xyz="${xyz}" rpy="0 0 0" />
+    </joint>
+  </xacro:macro>
+  <xacro:platform_joint pos="base" xyz="0 0 ${wheel_r + wheel_h_offset}" />
+  <xacro:platform_joint pos="upper" xyz="0 0 ${wheel_r + wheel_h_offset + 0.08}" />
   <!-- Stereo Camera -->
   <link name="camera_link">
     <visual>
       <geometry>
-        <box size="0.094 0.1168 0.071 "/>
+        <box size="0.020 0.075 0.015 "/>
       </geometry>
       <material name="black" />
@@ -49,5 +57,5 @@
     <parent link="base_link" />
     <child link="camera_link" />
-    <origin xyz="${platform_l / 2} 0 ${wheel_r + wheel_h_offset + 0.080}" rpy="0 0 0" />
+    <origin xyz="${platform_l / 2 + 0.01} 0 ${wheel_r + wheel_h_offset + 0.08}" rpy="0 0 0" />
   </joint>
 <!-- Differential Drive Wheels -->
@@ -103,5 +111,5 @@
   <xacro:macro name="sensor_joint" params="sensor pos rpy xyz">
     <joint name="${sensor}_${pos}_joint" type="fixed">
-      <parent link="platform" />
+      <parent link="platform_base" />
       <child link="${sensor}_${pos}" />
       <origin rpy="${rpy}" xyz="${xyz}" />

Commit message: updated urdf and xacro

File: urdf/mobile_base.urdf (robot description, URDF)
Before this commit: robot mobile_base, 16 links, 15 joints
Links:
- removed link camera_link
- added link left; visual box size=0.020 0.015 0.015
- added link right; visual box size=0.020 0.015 0.015
Joints:
- removed joint camera_base_link
- added joint camera_joint_left: type fixed, parent base_link, child left, origin xyz=0.1116 -0.053 0.0978 rpy=0 0 0
- added joint camera_joint_right: type fixed, parent base_link, child right, origin xyz=0.1116 0.053 0.0978 rpy=0 0 0

File: urdf/mobile_base.xacro (robot description, xacro)
@@ -46,17 +46,25 @@
   <xacro:platform_joint pos="upper" xyz="0 0 ${wheel_r + wheel_h_offset + 0.08}" />
   <!-- Stereo Camera -->
-  <link name="camera_link">
-    <visual>
-      <geometry>
-        <box size="0.020 0.075 0.015 "/>
-      </geometry>
-      <material name="black" />
-    </visual>
-  </link>
-  <joint name="camera_base_link" type="fixed">
-    <parent link="base_link" />
-    <child link="camera_link" />
-    <origin xyz="${platform_l / 2 + 0.01} 0 ${wheel_r + wheel_h_offset + 0.08}" rpy="0 0 0" />
-  </joint>
+  <xacro:macro name="camera" params="pos">
+    <link name="${pos}">
+      <visual>
+        <geometry>
+          <box size="0.020 0.015 0.015 "/>
+        </geometry>
+        <material name="black" />
+      </visual>
+    </link>
+  </xacro:macro>
+  <xacro:camera pos="left" />
+  <xacro:camera pos="right" />
+  <xacro:macro name="camera_joint" params="pos xyz">
+    <joint name="camera_joint_${pos}" type="fixed">
+      <parent link="base_link" />
+      <child link="${pos}" />
+      <origin xyz="${xyz}" rpy="0 0 0" />
+    </joint>
+  </xacro:macro>
+  <xacro:camera_joint pos="left" xyz="${platform_l / 2 + 0.01} -0.053 ${wheel_r + wheel_h_offset + 0.08}" />
+  <xacro:camera_joint pos="right" xyz="${platform_l / 2 + 0.01} 0.053 ${wheel_r + wheel_h_offset + 0.08}" />
 <!-- Differential Drive Wheels -->
   <xacro:macro name="wheel" params="pos rpy">

Commit message: rotate point cloud location

File: urdf/mobile_base.urdf (robot description, URDF)
Before this commit: robot mobile_base, 17 links, 16 joints
Joints:
- joint camera_joint_left: origin xyz=0.1116 -0.053 0.0978 rpy=0 0 0 -> xyz=0.1116 -0.053 0.0978 rpy=-1.5707963268 0 -1.5707963268
- joint camera_joint_right: origin xyz=0.1116 0.053 0.0978 rpy=0 0 0 -> xyz=0.1116 0.053 0.0978 rpy=-1.5707963268 0 -1.5707963268

File: urdf/mobile_base.xacro (robot description, xacro)
@@ -62,5 +62,5 @@
       <parent link="base_link" />
       <child link="${pos}" />
-      <origin xyz="${xyz}" rpy="0 0 0" />
+      <origin xyz="${xyz}" rpy="-${pi/2} 0 -${pi/2}" />
     </joint>
   </xacro:macro>
