Commit message: adding kinect instead of camera to urdf

File: urdf/mobile_base.urdf (robot description, URDF)
Before this commit: robot mobile_base, 17 links, 16 joints
Links:
- removed link left
- removed link right
- added link kinect_depth_frame, mass 0.0001
- added link kinect_depth_optical_frame, mass 0.0001
- added link kinect_link, mass 0.0001; visual box size=0.064 0.121 0.0381
Joints:
- removed joint camera_joint_left
- removed joint camera_joint_right
- added joint depth_optical_joint: type fixed, parent kinect_depth_frame, child kinect_depth_optical_frame, origin xyz=0 0 0 rpy=-1.5707963268 0 -1.5707963268
- added joint kinect_base_joint: type fixed, parent base_link, child kinect_link, origin xyz=0.1016 0 0.0978 rpy=0 0 0
- added joint kinect_depth_joint: type fixed, parent kinect_link, child kinect_depth_frame, origin xyz=0 0.028 0 rpy=0 0 0

File: urdf/mobile_base.xacro (robot description, xacro)
@@ -45,26 +45,52 @@
   <xacro:platform_joint pos="base" xyz="0 0 ${wheel_r + wheel_h_offset}" />
   <xacro:platform_joint pos="upper" xyz="0 0 ${wheel_r + wheel_h_offset + 0.08}" />
-  <!-- Stereo Camera -->
-  <xacro:macro name="camera" params="pos">
-    <link name="${pos}">
-      <visual>
-        <geometry>
-          <box size="0.020 0.015 0.015 "/>
-        </geometry>
-        <material name="black" />
-      </visual>
-    </link>
-  </xacro:macro>
-  <xacro:camera pos="left" />
-  <xacro:camera pos="right" />
-  <xacro:macro name="camera_joint" params="pos xyz">
-    <joint name="camera_joint_${pos}" type="fixed">
-      <parent link="base_link" />
-      <child link="${pos}" />
-      <origin xyz="${xyz}" rpy="-${pi/2} 0 -${pi/2}" />
-    </joint>
-  </xacro:macro>
-  <xacro:camera_joint pos="left" xyz="${platform_l / 2 + 0.01} -0.053 ${wheel_r + wheel_h_offset + 0.08}" />
-  <xacro:camera_joint pos="right" xyz="${platform_l / 2 + 0.01} 0.053 ${wheel_r + wheel_h_offset + 0.08}" />
+<link name="kinect_link">
+  <visual>
+    <geometry>
+      <box size="0.064 0.121 0.0381" />
+    </geometry>
+    <material name="Blue" />
+  </visual>
+  <inertial>
+      <mass value="0.0001" />
+      <origin xyz="0 0 0" />
+      <inertia ixx="0.0001" ixy="0.0" ixz="0.0"
+               iyy="0.0001" iyz="0.0"
+               izz="0.0001" />
+  </inertial>
+</link>
+<joint name="kinect_base_joint" type="fixed">
+  <origin xyz="${platform_l / 2} 0 ${wheel_r + wheel_h_offset + 0.08}" rpy="0 0 0" />
+  <parent link="base_link" />
+  <child link="kinect_link" />
+</joint>
+<joint name="kinect_depth_joint" type="fixed">
+  <origin xyz="0 0.028 0" rpy="0 0 0" />
+  <parent link="kinect_link" />
+  <child link="kinect_depth_frame" />
+</joint>
+<link name="kinect_depth_frame">
+  <inertial>
+      <mass value="0.0001" />
+      <origin xyz="0 0 0" />
+      <inertia ixx="0.0001" ixy="0.0" ixz="0.0"
+               iyy="0.0001" iyz="0.0"
+               izz="0.0001" />
+  </inertial>
+</link>
+<joint name="depth_optical_joint" type="fixed">
+  <origin xyz="0 0 0" rpy="-${pi/2} 0 -${pi/2}" />
+  <parent link="kinect_depth_frame" />
+  <child link="kinect_depth_optical_frame" />
+</joint>
+<link name="kinect_depth_optical_frame">
+  <inertial>
+      <mass value="0.0001" />
+      <origin xyz="0 0 0" />
+      <inertia ixx="0.0001" ixy="0.0" ixz="0.0"
+               iyy="0.0001" iyz="0.0"
+               izz="0.0001" />
+  </inertial>
+</link>
 <!-- Differential Drive Wheels -->
   <xacro:macro name="wheel" params="pos rpy">
@@ -156,2 +182,26 @@
   <xacro:sensor_depth_frame_joint sensor="ir" pos="right" />
 </robot>
+  <!-- Stereo Camera -->
+  <!--
+  <xacro:macro name="camera" params="pos">
+    <link name="${pos}">
+      <visual>
+        <geometry>
+          <box size="0.020 0.015 0.015 "/>
+        </geometry>
+        <material name="black" />
+      </visual>
+    </link>
+  </xacro:macro>
+  <xacro:camera pos="left" />
+  <xacro:camera pos="right" />
+  <xacro:macro name="camera_joint" params="pos xyz">
+    <joint name="camera_joint_${pos}" type="fixed">
+      <parent link="base_link" />
+      <child link="${pos}" />
+      <origin xyz="${xyz}" rpy="-${pi/2} 0 -${pi/2}" />
+    </joint>
+  </xacro:macro>
+  <xacro:camera_joint pos="left" xyz="${platform_l / 2 + 0.01} -0.053 ${wheel_r + wheel_h_offset + 0.08}" />
+  <xacro:camera_joint pos="right" xyz="${platform_l / 2 + 0.01} 0.053 ${wheel_r + wheel_h_offset + 0.08}" />
+  -->
