Commit message: updates to urdf to include imu and gps (fix) and include imu in rviz

File: urdf/head_unit.xacro (robot description, xacro)
@@ -17,45 +17,36 @@
     <origin xyz="0 0 1.2192" rpy="0 0 0" />
   </joint>
-  <!-- Bot platforms -->
-<!--
-  <xacro:macro name="platform" params="pos">
-    <link name="platform_${pos}">
-      <visual>
-        <geometry>
-          <box size="${platform_l} ${platform_w} ${platform_h}"/>
-        </geometry>
-        <material name="white">
-          <color rgba="1 1 1 1" />
-        </material>
-      </visual>
-    </link>
-  </xacro:macro>
-  <xacro:platform pos="base" />
-  <xacro:platform pos="upper" />
-  <xacro:macro name="platform_joint" params="pos xyz">
-    <joint name="platform_joint_${pos}" type="fixed">
-      <parent link="base_link" />
-      <child link="platform_${pos}" />
-      <origin xyz="${xyz}" rpy="0 0 0" />
-    </joint>
-  </xacro:macro>
-  <xacro:platform_joint pos="base" xyz="0 0 ${wheel_r + wheel_h_offset}" />
-  <xacro:platform_joint pos="upper" xyz="0 0 ${wheel_r + wheel_h_offset + 0.08}" />
-<link name="kinect_link">
-  <visual>
-    <geometry>
-      <box size="0.064 0.121 0.0381" />
-    </geometry>
-    <material name="Blue" />
-  </visual>
-  <inertial>
-      <mass value="0.0001" />
-      <origin xyz="0 0 0" />
-      <inertia ixx="0.0001" ixy="0.0" ixz="0.0"
-               iyy="0.0001" iyz="0.0"
-               izz="0.0001" />
-  </inertial>
-</link>
--->
+  <!-- IMU -->
+  <link name="imu">
+    <visual>
+      <geometry>
+        <box size="0.0001 0.0001 0.0001"/>
+      </geometry>
+      <material name="green">
+        <color rgba="0 192 0 1" />
+      </material>
+    </visual>
+  </link>
+  <joint name="head_unit_to_imu" type="fixed">
+    <parent link="head_unit" />
+    <child link="imu" />
+    <origin xyz="0 0 0" rpy="0 0 0" />
+  </joint>
+  <!-- GPS UNIT -->
+  <link name="fix">
+    <visual>
+      <geometry>
+        <box size="0.0001 0.0001 0.0001"/>
+      </geometry>
+      <material name="blue">
+        <color rgba="0 0 192 1" />
+      </material>
+    </visual>
+  </link>
+  <joint name="head_unit_to_fix" type="fixed">
+    <parent link="head_unit" />
+    <child link="fix" />
+    <origin xyz="0 0 0" rpy="0 0 0" />
+  </joint>
 <!--
 <node pkg="tf" type="static_transform_publisher" name="device_to_depth_cam" args="0 0 0 0 0.24 0 device depth_camera 10"/>

File: urdf/robot.urdf (robot description, URDF)
Before this commit: robot blah, 16 links, 15 joints
Links:
- added link fix; visual box size=0.0001 0.0001 0.0001
- added link imu; visual box size=0.0001 0.0001 0.0001
Joints:
- added joint head_unit_to_fix: type fixed, parent head_unit, child fix, origin xyz=0 0 0 rpy=0 0 0
- added joint head_unit_to_imu: type fixed, parent head_unit, child imu, origin xyz=0 0 0 rpy=0 0 0

Commit message: adding depth camera and fisheye camera to xacro and urdf

File: urdf/head_unit.xacro (robot description, xacro)
@@ -49,4 +49,34 @@
     <origin xyz="0 0 0" rpy="0 0 0" />
   </joint>
+  <link name="depth_camera">
+    <visual>
+      <geometry>
+        <box size="0.1 0.1 0.1"/>
+      </geometry>
+      <material name="blue">
+        <color rgba="0 0 192 1" />
+      </material>
+    </visual>
+  </link>
+  <joint name="head_unit_to_depth_camera" type="fixed">
+    <parent link="head_unit" />
+    <child link="depth_camera" />
+    <origin xyz="0 0.24 0" rpy="0 0 0" />
+  </joint>
+  <link name="fisheye_camera">
+    <visual>
+      <geometry>
+        <box size="0.1 0.1 0.1"/>
+      </geometry>
+      <material name="red">
+        <color rgba="192 0 0 1" />
+      </material>
+    </visual>
+  </link>
+  <joint name="head_unit_to_fisheye_camera" type="fixed">
+    <parent link="head_unit" />
+    <child link="fisheye_camera" />
+    <origin xyz="0 0.24 0" rpy="0 0 0" />
+  </joint>
 <!--
 <node pkg="tf" type="static_transform_publisher" name="device_to_depth_cam" args="0 0 0 0 0.24 0 device depth_camera 10"/>

File: urdf/robot.urdf (robot description, URDF)
Before this commit: robot blah, 18 links, 17 joints
Links:
- added link depth_camera; visual box size=0.1 0.1 0.1
- added link fisheye_camera; visual box size=0.1 0.1 0.1
Joints:
- added joint head_unit_to_depth_camera: type fixed, parent head_unit, child depth_camera, origin xyz=0 0.24 0 rpy=0 0 0
- added joint head_unit_to_fisheye_camera: type fixed, parent head_unit, child fisheye_camera, origin xyz=0 0.24 0 rpy=0 0 0

Commit message: set fisheye and depth camera apart from each other, easier to see

File: urdf/head_unit.xacro (robot description, xacro)
@@ -77,5 +77,5 @@
     <parent link="head_unit" />
     <child link="fisheye_camera" />
-    <origin xyz="0 0.24 0" rpy="0 0 0" />
+    <origin xyz="0 0.4 0" rpy="0 0 0" />
   </joint>
 <!--

File: urdf/robot.urdf (robot description, URDF)
Before this commit: robot blah, 20 links, 19 joints
Joints:
- joint head_unit_to_fisheye_camera: origin xyz=0 0.24 0 rpy=0 0 0 -> xyz=0 0.4 0 rpy=0 0 0

Commit message: add image proc to get rectified images, add point cloud converter

File: urdf/head_unit.xacro (robot description, xacro)
@@ -52,5 +52,5 @@
     <visual>
       <geometry>
-        <box size="0.1 0.1 0.1"/>
+        <box size="0.05 0.05 0.05"/>
       </geometry>
       <material name="blue">
@@ -67,5 +67,5 @@
     <visual>
       <geometry>
-        <box size="0.1 0.1 0.1"/>
+        <box size="0.05 0.05 0.05"/>
       </geometry>
       <material name="red">

File: urdf/robot.urdf (robot description, URDF)
Before this commit: robot blah, 20 links, 19 joints
Links:
- link depth_camera: geometry visual box size=0.05 0.05 0.05
- link fisheye_camera: geometry visual box size=0.05 0.05 0.05
