Commit message: Adding urdf for gps.

File: urdf/mower.urdf (robot description, URDF)
Before this commit: robot mower, 7 links, 6 joints
Links:
- added link gps; visual box size=0.025 0.025 0.0125
Joints:
- added joint gps_joint: type fixed, parent base_link, child gps, origin xyz=0 0 .4

File: urdf/mower.xacro (robot description, xacro)
@@ -99,3 +99,17 @@
     <origin xyz="0.336 0 -${(platform_h / 2) - 0.1 + 0.025}" />
   </joint>
+<!-- GPS -->
+  <link name="gps">
+    <visual>
+      <geometry>
+        <box size="0.025 0.025 0.0125" />
+      </geometry>
+      <material name="white" />
+    </visual>
+  </link>
+  <joint name="gps_joint" type="fixed">
+    <parent link="base_link" />
+    <child link="gps" />
+    <origin xyz="0 0 .4" />
+  </joint>
 </robot>
